Commit message: change mass and inertia

File: urdf/antsy_description.xacro (robot description, xacro)
@@ -23,9 +23,8 @@
     </collision>
     <inertial>
-      <mass value="0.300" />
-      <origin xyz="0 0 0" />
-      <inertia ixx="0.0021" iyy="0.0046" izz="0.0065"
-               ixy="0" ixz="0" iyz="0" />
-    </inertial>
+    <origin xyz="0.00014120578374947324 0.000907462590201314 -0.0004863329579636028" rpy="0 0 0"/>
+    <mass value="0.9"/> <!-- changed from  6.980366975019921 -->
+    <inertia ixx="0.035507" ixy="8e-06" ixz="-1.7e-05" iyy="0.050259" iyz="4e-06" izz="0.082758"/>
+  </inertial>
   </link>
   <!-- legs -->
@@ -70,8 +69,7 @@
       </collision>
       <inertial>
-        <mass value="0.100" />
+        <mass value="0.09" /> <!-- changed from 0.06644962989519385 -->
         <origin xyz="${leg_a_length/2} 0 0" />
-        <inertia ixx="0.000028" iyy="0.000028" izz="0.000028"
-                 ixy="0"        ixz="0"        iyz="0" />
+            <inertia ixx="3.4e-05" iyy="3.2e-05" izz="2.4e-05" ixy="-0.0" iyz="0.0" ixz="-0.0"/>
       </inertial>
     </link>
@@ -100,8 +98,7 @@
       </collision>
       <inertial>
-        <mass value="0.100" />
+        <mass value="0.08" /> <!-- changed from 0.029822153915739318 -->
         <origin xyz="${leg_b_length/2} 0 0" />
-        <inertia ixx="0.000195" iyy="0.000010" izz="0.000195"
-                 ixy="0"        ixz="0"        iyz="0" />
+        <inertia ixx="2.7e-05" iyy="1.9e-05" izz="4.1e-05" ixy="0.0" iyz="-1e-06" ixz="-0.0"/>
       </inertial>
     </link>
@@ -145,8 +142,7 @@
       </collision>
       <inertial>
-        <mass value="0.100" />
+        <mass value="0.030" /> <!-- changed from 0.08076187945098641 -->
         <origin xyz="${leg_c_length/2} 0 0" rpy="0 -0.35 0" />
-        <inertia ixx="0.000195" iyy="0.000010" izz="0.000195"
-                 ixy="0"        ixz="0"        iyz="0" />
+        <inertia ixx="0.000205" iyy="3.9e-05" izz="0.000199" ixy="2e-06" iyz="4.1e-05" ixz="-0.0"/>
       </inertial>
     </link>

Commit message: update xacro to match the real robot joint directions

File: urdf/antsy_description.xacro (robot description, xacro)
@@ -45,5 +45,5 @@
     </gazebo>
   </xacro:macro>
-  <xacro:macro name="leg" params="index reflect xyz rpy">
+  <xacro:macro name="leg" params="index reflect_coxa reflect_tibia reflect_foot xyz rpy">
     <!-- leg_X: fixed to base_link -->
     <link name="leg_${index}" />
@@ -75,7 +75,7 @@
     </link>
     <joint name="leg_${index}_base__leg_${index}a" type="revolute">
-      <axis xyz="0 0 1" />
+      <axis xyz="0 0 ${reflect_coxa}" />
       <limit lower="${joint_a_limit_lower}" upper="${joint_a_limit_upper}"
-          effort="${servo_effort_limit}" velocity="${servo_velocity_limit}" />
+        effort="${servo_effort_limit}" velocity="${servo_velocity_limit}" />
       <parent link="leg_${index}" />
       <child link="leg_${index}a" />
@@ -104,5 +104,5 @@
     </link>
     <joint name="leg_${index}a__leg_${index}b" type="revolute">
-      <axis xyz="0 1 0" />
+      <axis xyz="0 ${reflect_tibia} 0" />
       <limit lower="${joint_b_limit_lower}" upper="${joint_b_limit_upper}"
         effort="${servo_effort_limit}" velocity="${servo_velocity_limit}" />
@@ -148,5 +148,5 @@
     </link>
     <joint name="leg_${index}b__leg_${index}c" type="revolute">
-      <axis xyz="0 1 0" />
+      <axis xyz="0 ${reflect_foot} 0" />
       <limit lower="${joint_c_limit_lower}" upper="${joint_c_limit_upper}"
         effort="${servo_effort_limit}" velocity="${servo_velocity_limit}" />
@@ -168,10 +168,10 @@
   </xacro:macro>
   <!-- Instantiate the six legs -->
-  <xacro:leg index="0" reflect="1"  xyz=" 0.138  0.0875 0.0" rpy="0 0 ${pi/2 - leg_spreading_angle}" />
-  <xacro:leg index="1" reflect="1"  xyz=" 0.00  0.11950 0.0" rpy="0 0 ${pi/2}" />
-  <xacro:leg index="2" reflect="1"  xyz="-0.138  0.0875 0.0" rpy="0 0 ${pi/2 + leg_spreading_angle}" />
-  <xacro:leg index="3" reflect="-1" xyz="-0.138 -0.0875 0.0" rpy="0 0 ${-pi/2 -leg_spreading_angle}" />
-  <xacro:leg index="4" reflect="-1" xyz=" 0.00 -0.11950 0.0" rpy="0 0 ${-pi/2}" />
-  <xacro:leg index="5" reflect="-1" xyz=" 0.138 -0.0875 0.0" rpy="0 0 ${-pi/2 + leg_spreading_angle}" />
+  <xacro:leg index="0" reflect_coxa="1" reflect_tibia="-1" reflect_foot="1" xyz=" 0.138  0.0875 0.0" rpy="0 0 ${pi/2 - leg_spreading_angle}" />
+  <xacro:leg index="1" reflect_coxa="1" reflect_tibia="-1" reflect_foot="1"  xyz=" 0.00  0.11950 0.0" rpy="0 0 ${pi/2}" />
+  <xacro:leg index="2" reflect_coxa="1" reflect_tibia="-1" reflect_foot="1"  xyz="-0.138  0.0875 0.0" rpy="0 0 ${pi/2 + leg_spreading_angle}" />
+  <xacro:leg index="3" reflect_coxa="1" reflect_tibia="1" reflect_foot="-1" xyz="-0.138 -0.0875 0.0" rpy="0 0 ${-pi/2 -leg_spreading_angle}" />
+  <xacro:leg index="4" reflect_coxa="1" reflect_tibia="1" reflect_foot="-1" xyz=" 0.00 -0.11950 0.0" rpy="0 0 ${-pi/2}" />
+  <xacro:leg index="5" reflect_coxa="1" reflect_tibia="1" reflect_foot="-1" xyz=" 0.138 -0.0875 0.0" rpy="0 0 ${-pi/2 + leg_spreading_angle}" />
   <!-- Sensors -->
   <link name="imu" />

Commit message: make robot description work in gazebo

File: urdf/antsy_description.xacro (robot description, xacro)
@@ -64,5 +64,5 @@
       </visual>
       <collision>
-        <origin xyz="${leg_a_length/2} 0.05 0.05"/>
+        <origin xyz="${leg_a_length/2} 0.0 0.0"/>
         <geometry>
           <box size="${leg_a_length} 0.05 0.05" />
@@ -194,6 +194,6 @@
       <odom_publish_frequency>50</odom_publish_frequency>
       <odom_topic>/antsy/odometry</odom_topic>
-      <odom_frame>world</odom_frame>
-      <robot_base_frame>base_link</robot_base_frame>
+      <odom_frame>odom</odom_frame>
+      <robot_base_frame>base_footprint</robot_base_frame>
     </plugin>
     <plugin

File: urdf/properties.urdf.xacro (robot description, xacro)
@@ -17,5 +17,8 @@
   <xacro:property name="leg_b_length" value="0.100" />
   <xacro:property name="leg_c_length" value="0.150" />
-  <xacro:property name="servo_velocity_limit" value="5.6" /> <!-- datasheet tells 5.81 -->
+  <!-- datasheet tells 5.81 -->
+  <!-- <xacro:property name="servo_velocity_limit" value="5.6" /> -->
+  <!-- debug setting -->
+  <xacro:property name="servo_velocity_limit" value="110.2" />
   <xacro:property name="servo_effort_limit" value="4.25" /> <!-- datasheet tells 4.0-4.4 -->
   <xacro:property name="servo_static_friction" value="0.3" />

Commit message: save local changes in temp branch

File: urdf/antsy_description.xacro (robot description, xacro)
@@ -23,9 +23,8 @@
     </collision>
     <inertial>
-      <mass value="0.300" />
-      <origin xyz="0 0 0" />
-      <inertia ixx="0.0021" iyy="0.0046" izz="0.0065"
-               ixy="0" ixz="0" iyz="0" />
-    </inertial>
+    <origin xyz="0.00014120578374947324 0.000907462590201314 -0.0004863329579636028" rpy="0 0 0"/>
+    <mass value="0.9"/> <!-- changed from  6.980366975019921 -->
+    <inertia ixx="0.035507" ixy="8e-06" ixz="-1.7e-05" iyy="0.050259" iyz="4e-06" izz="0.082758"/>
+  </inertial>
   </link>
   <!-- legs -->
@@ -46,5 +45,5 @@
     </gazebo>
   </xacro:macro>
-  <xacro:macro name="leg" params="index reflect xyz rpy">
+  <xacro:macro name="leg" params="index reflect_coxa reflect_tibia reflect_foot xyz rpy">
     <!-- leg_X: fixed to base_link -->
     <link name="leg_${index}" />
@@ -64,5 +63,5 @@
       </visual>
       <collision>
-        <origin xyz="${leg_a_length/2} 0.0 0.0"/>
+        <origin xyz="${leg_a_length/2} 0.05 0.05"/>
         <geometry>
           <box size="${leg_a_length} 0.05 0.05" />
@@ -70,14 +69,13 @@
       </collision>
       <inertial>
-        <mass value="0.100" />
+        <mass value="0.09" /> <!-- changed from 0.06644962989519385 -->
         <origin xyz="${leg_a_length/2} 0 0" />
-        <inertia ixx="0.000028" iyy="0.000028" izz="0.000028"
-                 ixy="0"        ixz="0"        iyz="0" />
+            <inertia ixx="3.4e-05" iyy="3.2e-05" izz="2.4e-05" ixy="-0.0" iyz="0.0" ixz="-0.0"/>
       </inertial>
     </link>
     <joint name="leg_${index}_base__leg_${index}a" type="revolute">
-      <axis xyz="0 0 1" />
+      <axis xyz="0 0 ${reflect_coxa}" />
       <limit lower="${joint_a_limit_lower}" upper="${joint_a_limit_upper}"
-          effort="${servo_effort_limit}" velocity="${servo_velocity_limit}" />
+        effort="${servo_effort_limit}" velocity="${servo_velocity_limit}" />
       <parent link="leg_${index}" />
       <child link="leg_${index}a" />
@@ -100,12 +98,11 @@
       </collision>
       <inertial>
-        <mass value="0.100" />
+        <mass value="0.08" /> <!-- changed from 0.029822153915739318 -->
         <origin xyz="${leg_b_length/2} 0 0" />
-        <inertia ixx="0.000195" iyy="0.000010" izz="0.000195"
-                 ixy="0"        ixz="0"        iyz="0" />
+        <inertia ixx="2.7e-05" iyy="1.9e-05" izz="4.1e-05" ixy="0.0" iyz="-1e-06" ixz="-0.0"/>
       </inertial>
     </link>
     <joint name="leg_${index}a__leg_${index}b" type="revolute">
-      <axis xyz="0 1 0" />
+      <axis xyz="0 ${reflect_tibia} 0" />
       <limit lower="${joint_b_limit_lower}" upper="${joint_b_limit_upper}"
         effort="${servo_effort_limit}" velocity="${servo_velocity_limit}" />
@@ -145,12 +142,11 @@
       </collision>
       <inertial>
-        <mass value="0.100" />
+        <mass value="0.030" /> <!-- changed from 0.08076187945098641 -->
         <origin xyz="${leg_c_length/2} 0 0" rpy="0 -0.35 0" />
-        <inertia ixx="0.000195" iyy="0.000010" izz="0.000195"
-                 ixy="0"        ixz="0"        iyz="0" />
+        <inertia ixx="0.000205" iyy="3.9e-05" izz="0.000199" ixy="2e-06" iyz="4.1e-05" ixz="-0.0"/>
       </inertial>
     </link>
     <joint name="leg_${index}b__leg_${index}c" type="revolute">
-      <axis xyz="0 1 0" />
+      <axis xyz="0 ${reflect_foot} 0" />
       <limit lower="${joint_c_limit_lower}" upper="${joint_c_limit_upper}"
         effort="${servo_effort_limit}" velocity="${servo_velocity_limit}" />
@@ -172,10 +168,10 @@
   </xacro:macro>
   <!-- Instantiate the six legs -->
-  <xacro:leg index="0" reflect="1"  xyz=" 0.138  0.0875 0.0" rpy="0 0 ${pi/2 - leg_spreading_angle}" />
-  <xacro:leg index="1" reflect="1"  xyz=" 0.00  0.11950 0.0" rpy="0 0 ${pi/2}" />
-  <xacro:leg index="2" reflect="1"  xyz="-0.138  0.0875 0.0" rpy="0 0 ${pi/2 + leg_spreading_angle}" />
-  <xacro:leg index="3" reflect="-1" xyz="-0.138 -0.0875 0.0" rpy="0 0 ${-pi/2 -leg_spreading_angle}" />
-  <xacro:leg index="4" reflect="-1" xyz=" 0.00 -0.11950 0.0" rpy="0 0 ${-pi/2}" />
-  <xacro:leg index="5" reflect="-1" xyz=" 0.138 -0.0875 0.0" rpy="0 0 ${-pi/2 + leg_spreading_angle}" />
+  <xacro:leg index="0" reflect_coxa="1" reflect_tibia="-1" reflect_foot="1" xyz=" 0.138  0.0875 0.0" rpy="0 0 ${pi/2 - leg_spreading_angle}" />
+  <xacro:leg index="1" reflect_coxa="1" reflect_tibia="-1" reflect_foot="1"  xyz=" 0.00  0.11950 0.0" rpy="0 0 ${pi/2}" />
+  <xacro:leg index="2" reflect_coxa="1" reflect_tibia="-1" reflect_foot="1"  xyz="-0.138  0.0875 0.0" rpy="0 0 ${pi/2 + leg_spreading_angle}" />
+  <xacro:leg index="3" reflect_coxa="1" reflect_tibia="1" reflect_foot="-1" xyz="-0.138 -0.0875 0.0" rpy="0 0 ${-pi/2 -leg_spreading_angle}" />
+  <xacro:leg index="4" reflect_coxa="1" reflect_tibia="1" reflect_foot="-1" xyz=" 0.00 -0.11950 0.0" rpy="0 0 ${-pi/2}" />
+  <xacro:leg index="5" reflect_coxa="1" reflect_tibia="1" reflect_foot="-1" xyz=" 0.138 -0.0875 0.0" rpy="0 0 ${-pi/2 + leg_spreading_angle}" />
   <!-- Sensors -->
   <link name="imu" />
@@ -194,6 +190,6 @@
       <odom_publish_frequency>50</odom_publish_frequency>
       <odom_topic>/antsy/odometry</odom_topic>
-      <odom_frame>odom</odom_frame>
-      <robot_base_frame>base_footprint</robot_base_frame>
+      <odom_frame>world</odom_frame>
+      <robot_base_frame>base_link</robot_base_frame>
     </plugin>
     <plugin

Commit message: Wire Gazebo joint position controllers

File: urdf/antsy_description.xacro (robot description, xacro)
@@ -29,5 +29,5 @@
   </link>
   <!-- legs -->
-  <xacro:macro name="servo" params="index joint_name">
+  <xacro:macro name="servo" params="joint_name">
     <gazebo>
       <plugin
@@ -35,6 +35,5 @@
         name="gz::sim::systems::JointPositionController">
         <joint_name>${joint_name}</joint_name>
-        <use_actuator_msg>true</use_actuator_msg>
-        <actuator_number>${index}</actuator_number>
+        <topic>/antsy/joint_position/${joint_name}</topic>
         <cmd_max>${servo_effort_limit}</cmd_max>
         <cmd_min>${-servo_effort_limit}</cmd_min>
@@ -163,7 +162,7 @@
       <origin xyz="${leg_c_length} 0 0" rpy="0 0.4 0"/>
     </joint>
-    <xacro:servo index="${index*3+0}" joint_name="leg_${index}_base__leg_${index}a" />
-    <xacro:servo index="${index*3+1}" joint_name="leg_${index}a__leg_${index}b" />
-    <xacro:servo index="${index*3+2}" joint_name="leg_${index}b__leg_${index}c" />
+    <xacro:servo joint_name="leg_${index}_base__leg_${index}a" />
+    <xacro:servo joint_name="leg_${index}a__leg_${index}b" />
+    <xacro:servo joint_name="leg_${index}b__leg_${index}c" />
   </xacro:macro>
   <!-- Instantiate the six legs -->

File: urdf/properties.urdf.xacro (robot description, xacro)
@@ -13,16 +13,18 @@
   <!-- Parameters -->
   <!-- ********** -->
+  <xacro:arg name="servo_velocity_limit" default="5.6" />
+  <xacro:arg name="servo_effort_limit" default="4.25" />
+  <xacro:arg name="servo_static_friction" default="0.3" />
+  <xacro:arg name="servo_damping_friction" default="0.1" />
+  <xacro:arg name="servo_p_gain" default="17.8" />
   <xacro:property name="leg_spreading_angle" value="1.0472" />
   <xacro:property name="leg_a_length" value="0.04375" />
   <xacro:property name="leg_b_length" value="0.100" />
   <xacro:property name="leg_c_length" value="0.150" />
-  <!-- datasheet tells 5.81 -->
-  <!-- <xacro:property name="servo_velocity_limit" value="5.6" /> -->
-  <!-- debug setting -->
-  <xacro:property name="servo_velocity_limit" value="110.2" />
-  <xacro:property name="servo_effort_limit" value="4.25" /> <!-- datasheet tells 4.0-4.4 -->
-  <xacro:property name="servo_static_friction" value="0.3" />
-  <xacro:property name="servo_damping_friction" value="0.1" />
-  <xacro:property name="servo_p_gain" value="17.8" />
+  <xacro:property name="servo_velocity_limit" value="$(arg servo_velocity_limit)" />
+  <xacro:property name="servo_effort_limit" value="$(arg servo_effort_limit)" />
+  <xacro:property name="servo_static_friction" value="$(arg servo_static_friction)" />
+  <xacro:property name="servo_damping_friction" value="$(arg servo_damping_friction)" />
+  <xacro:property name="servo_p_gain" value="$(arg servo_p_gain)" />
   <xacro:property name="joint_a_limit_lower" value="-1.5708" />
   <xacro:property name="joint_a_limit_upper" value="1.5708" />

Commit message: Remove Gazebo-specific description hooks

File: urdf/antsy_description.xacro (robot description, xacro)
@@ -29,19 +29,4 @@
   </link>
   <!-- legs -->
-  <xacro:macro name="servo" params="joint_name">
-    <gazebo>
-      <plugin
-        filename="gz-sim-joint-position-controller-system"
-        name="gz::sim::systems::JointPositionController">
-        <joint_name>${joint_name}</joint_name>
-        <topic>/antsy/joint_position/${joint_name}</topic>
-        <cmd_max>${servo_effort_limit}</cmd_max>
-        <cmd_min>${-servo_effort_limit}</cmd_min>
-        <p_gain>${servo_p_gain}</p_gain>
-        <i_gain>0.</i_gain>
-        <d_gain>0.</d_gain>
-      </plugin>
-    </gazebo>
-  </xacro:macro>
   <xacro:macro name="leg" params="index reflect_coxa reflect_tibia reflect_foot xyz rpy">
     <!-- leg_X: fixed to base_link -->
@@ -162,7 +147,4 @@
       <origin xyz="${leg_c_length} 0 0" rpy="0 0.4 0"/>
     </joint>
-    <xacro:servo joint_name="leg_${index}_base__leg_${index}a" />
-    <xacro:servo joint_name="leg_${index}a__leg_${index}b" />
-    <xacro:servo joint_name="leg_${index}b__leg_${index}c" />
   </xacro:macro>
   <!-- Instantiate the six legs -->
@@ -181,26 +163,3 @@
     <origin xyz="0 0 0.05" />
   </joint>
-  <!-- Gazebo (simulation only) -->
-  <!-- docs: https://github.com/gazebosim/gz-sim/tree/main/src/systems -->
-  <gazebo>
-    <plugin
-      filename="gz-sim-odometry-publisher-system"
-      name="gz::sim::systems::OdometryPublisher">
-      <odom_publish_frequency>50</odom_publish_frequency>
-      <odom_topic>/antsy/odometry</odom_topic>
-      <odom_frame>odom</odom_frame>
-      <robot_base_frame>base_footprint</robot_base_frame>
-    </plugin>
-    <plugin
-      filename="gz-sim-joint-state-publisher-system"
-      name="gz::sim::systems::JointStatePublisher">
-      <topic>/antsy/joint_state</topic>
-    </plugin>
-    <!-- TODO doesn't work, no imu topic in Gazebo gets published -->
-    <plugin
-      filename="gz-sim-imu-system"
-      name="gz::sim::systems::Imu">
-      <topic>/antsy/imu</topic>
-    </plugin>
-  </gazebo>
 </robot>

File: urdf/properties.urdf.xacro (robot description, xacro)
@@ -17,5 +17,4 @@
   <xacro:arg name="servo_static_friction" default="0.3" />
   <xacro:arg name="servo_damping_friction" default="0.1" />
-  <xacro:arg name="servo_p_gain" default="17.8" />
   <xacro:property name="leg_spreading_angle" value="1.0472" />
   <xacro:property name="leg_a_length" value="0.04375" />
@@ -26,5 +25,4 @@
   <xacro:property name="servo_static_friction" value="$(arg servo_static_friction)" />
   <xacro:property name="servo_damping_friction" value="$(arg servo_damping_friction)" />
-  <xacro:property name="servo_p_gain" value="$(arg servo_p_gain)" />
   <xacro:property name="joint_a_limit_lower" value="-1.5708" />
   <xacro:property name="joint_a_limit_upper" value="1.5708" />
